File: hardware/stm32-network-rs232.sch (KiCad schematic (older format))
At the start: 0 parts

Commit message: update libs
Parts:
- added C101, C102: 18pF, symbol C
- added C103, C104: 47pF, symbol C
- added C105, C106, C107, C108, C109: C, symbol C
- added J101: USB, symbol USB
- added M101, M102, M103, M104: Mount Hole, symbol MECH
- added P101: DEBUG, symbol FTDI-PLUG
- added P?: SWD, symbol SWD
- added P?: RS232-TAP, symbol FTDI-PLUG
- added R101: 10K, symbol R
- added R102, R103: 22R, symbol R
- added R104: 1.5K, symbol R
- added U101: MOSFET-P, symbol MOSFET-P
- added U102: STM32-48PIN, symbol STM32-48PIN
- added X101: 8MHz, symbol CRYSTAL
Connections:
- new net: C101.1, U102.5 (PD0/OSCIN), X101.1
- new net: C102.1, U102.6 (PD1/OSCOUT), X101.2
- new net: J101.2 (D-), R102.2
- new net: J101.3 (D+), R103.2
- new net: R104.2, U101.2
- new net +3.3V: C105.2, C106.2, C107.2, C108.2, C109.2, J101.1 (VBUS), P?.1 (VDD_TARGET), R101.2, U101.3, U102.1 (Vbat), U102.24 (Vdd), U102.36 (Vdd), U102.48 (Vdd), U102.9 (Vdda)
- new net GNDPWR: C101.2, C102.2, C103.2, C104.2, C105.1, C106.1, C107.1, C108.1, C109.1, J101.5 (GND), J101.6 (SHIELD), P101.1 (GND/BLACK), P?.1 (GND/BLACK), P?.3 (GND), U102.23 (Vss), U102.35 (Vss), U102.44 (BOOT0), U102.47 (Vss), U102.8 (Vssa)
- new net SWCLK: P?.2 (SWCLK), U102.37 (PA14/JTCK/SWCLK)
- new net SWDIO: P?.4 (SWDIO), U102.34 (PA13/JTMS-SWDIO)
- new net USART1RX: P101.4 (TXD/ORANGE), U102.31 (PA10/USART1RX)
- new net USART1TX: P101.5 (RXD/YELLOW), U102.30 (PA9/USART1TX)
- new net USART2RX: P?.4 (TXD/ORANGE), U102.13 (PA3/USART2RX/ADCIN3/TIM2CH4)
- new net USART2TX: P?.5 (RXD/YELLOW), U102.12 (PA2/USART2TX/ADCIN2/TIM2CH3)
- new net USBDIS: R101.1, U101.1, U102.29 (PA8/USART1CK/MCO)
- new net USBDM: C104.1, R102.1, U102.32 (PA11/USART1CTS/USBDM)
- new net USBDP: C103.1, R103.1, R104.1, U102.33 (PA12/USART1RTS/USBDP)
- new net nRST: P?.5 (NRST), U102.7 (~RST)
- no-connect marks 0 -> 9
Other:
- note added: "Flash Memory\nBOOT0=0 BOOT1=X"
- note added: "RST has internal pull-up"
