File: hardware/stm32-network-rs232.sch (KiCad schematic (older format))
At the start: 57 parts, among them J1 USB, M1 Mount Hole, M2 Mount Hole, M3 Mount Hole, M4 Mount Hole, P1 BELFUSE-08B0-1X1T-06-F, P2 P10, P3 DEBUG, P4 SWD, P5 RS232-TAP, P6 RS-232-DB-9-DTE, P7 P03, P8 P03, U1 ENC28J60, U2 STM32-48PIN, U3 MAX3221, U4 MOSFET-P, U5 ZLDO1117, X1 25MHz, X2 8MHz

Commit message: removed utils, added contiki
Parts:
- U2: value STM32-48PIN -> STM32F103CBT6
Changed lines of the file:
@@
 P 4050 2500
 F 0 "U2" H 3050 4250 60  0000 C CNN
-F 1 "STM32-48PIN" H 3700 750 60  0000 C CNN
+F 1 "STM32F103CBT6" H 3700 750 60  0000 C CNN
 F 2 "kicad-new-lib:QFP50P900X900X160-48N" H 4050 2500 60  0001 C CNN
 F 3 "" H 4050 2500 60  0000 C CNN
